Commit message: update speed

File: ros2_ws/ros_cassandra_description/urdf/control_cassandra.xacro (robot description, xacro)
@@ -2,5 +2,6 @@
 <robot xmlns:xacro="http://www.ros.org/wiki/xacro">
     <xacro:arg name="dc_motor_dry_run" default="false"/>
-    <xacro:property name="max_wheel_speed_rad_s" value="16.6666666667"/>
+    <!-- 3.0 m/s / 0.03 m wheel radius = 100 rad/s -->
+    <xacro:property name="max_wheel_speed_rad_s" value="100.0"/>
     <ros2_control name="CassandraBaseHardware" type="system">
         <hardware>
@@ -10,5 +11,5 @@
             <param name="pwm_frequency">1000</param>
             <param name="min_pwm_percent">8.0</param>
-            <param name="max_pwm_percent">15.0</param>
+            <param name="max_pwm_percent">100.0</param>
             <param name="max_wheel_speed_rad_s">${max_wheel_speed_rad_s}</param>
             <param name="command_deadband_rad_s">0.05</param>
